Commit message: testing

File: calypso_sim/model/chasis.urdf.xacro (robot description, xacro)
@@ -17,6 +17,7 @@
     </collision>
     <inertial>
-      <mass value="37"/>
+      <mass value="370"/>
       <inertia ixx="1002084.26190628" ixy="-0.00000934" ixz="-0.00004849" iyy="1472890.49211890" iyz="1402.25179064" izz="689649.10160904"/>
+      <!-- <inertia ixx="0" ixy="0.0" ixz="0.0" iyy="0" iyz="0" izz="0"/> -->
     </inertial>
   </link>

Commit message: rolling back

File: calypso_sim/model/chasis.urdf.xacro (robot description, xacro)
@@ -16,8 +16,11 @@
       <origin xyz="${xyz}" rpy="${rpy}"/>
     </collision>
+    <!-- <inertial>
+      <mass value="37"/>
+      <inertia ixx="1002084.26190628" ixy="-0.00000934" ixz="-0.00004849" iyy="1472890.49211890" iyz="1402.25179064" izz="689649.10160904"/>
+    </inertial> -->
     <inertial>
-      <mass value="370"/>
-      <inertia ixx="1002084.26190628" ixy="-0.00000934" ixz="-0.00004849" iyy="1472890.49211890" iyz="1402.25179064" izz="689649.10160904"/>
-      <!-- <inertia ixx="0" ixy="0.0" ixz="0.0" iyy="0" iyz="0" izz="0"/> -->
+      <mass value="37"/>
+      <inertia ixx="-0.00000934" ixy="-0.00000934" ixz="-0.00000934" iyy="-0.00000934" iyz="-0.00000934" izz="-0.00000934"/>
     </inertial>
   </link>

Commit message: pushing production testing

File: calypso_sim/model/chasis.urdf.xacro (robot description, xacro)
@@ -21,6 +21,6 @@
     </inertial> -->
     <inertial>
-      <mass value="37"/>
-      <inertia ixx="-0.00000934" ixy="-0.00000934" ixz="-0.00000934" iyy="-0.00000934" iyz="-0.00000934" izz="-0.00000934"/>
+      <mass value="38.00000000"/>
+      <inertia ixx="1029167.62033618" ixy="-0.00000959" ixz="-0.00004980" iyy="1512698.34325725" iyz="1440.15048769" izz="708288.26651739"/>
     </inertial>
   </link>
