Commit message: modified for camera and imu

File: calypso_sim/model/auv.urdf.xacro (robot description, xacro)
@@ -2,5 +2,5 @@
 <robot xmlns:xacro="http://www.ros.org/wiki/xacro" name="auv">
     <xacro:include filename="$(find calypso_sim)/model/camera.urdf.xacro"/>
-    <!-- <xacro:include filename="$(find calypso_sim)/model/imu.urdf.xacro"/> -->
+    <xacro:include filename="$(find calypso_sim)/model/imu.urdf.xacro"/>
     <xacro:include filename="$(find calypso_sim)/model/thrusters.urdf.xacro"/>
     <material name="red">
@@ -77,8 +77,8 @@
     <xacro:thruster_CW id="8" parent="base_link" xyz="-0.23 -0.23 0.06" rpy="0 1.57 2.182" axis="0 0 1">
     </xacro:thruster_CW>
-    <xacro:camera id="1" parent="base_link" xyz="0.3 -0.55 0.19" rpy="0 0 -1.57">
+    <xacro:camera id="1" parent="base_link" xyz="-0.02 -0.2 0.19" rpy="0 0 -1.57">
     </xacro:camera>
-    <!-- <xacro:imu id="1" parent="base_link" xyz="0.3 -0.55 0.19" rpy="0 0 -1.57">
-    </xacro:imu> -->
+    <xacro:imu id="1" parent="base_link" xyz="-0.02 0.1 0.06" rpy="0 0 -1.57">
+    </xacro:imu>
     <gazebo>
       <plugin name="gazebo_ros_control" filename="libgazebo_ros_control.so">

File: calypso_sim/model/imu.urdf.xacro (robot description, xacro)
@@ -11,5 +11,5 @@
                 <origin xyz="0 0 0" rpy="0 0 0"/>
                 <geometry>
-                    <box size="0.01 0.01 0.01"/>
+                    <box size="0.1 0.1 0.1"/>
                 </geometry>
             </collision>
@@ -17,5 +17,5 @@
                 <origin xyz="0 0 0" rpy="0 0 0"/>
                 <geometry>
-                    <box size="0.01 0.01 0.01"/>
+                    <box size="0.1 0.1 0.1"/>
                 </geometry>
                 <material name="blue"/>
@@ -28,11 +28,11 @@
         </link>
         <gazebo reference="imu_${id}_link">
-            <plugin name="imu_plugin" filename="libgazebo_ros_imu.so">
-            <alwaysOn>true</alwaysOn>
-            <bodyName>base_footprint</bodyName>
-            <topicName>imu</topicName>
-            <serviceName>imu_service</serviceName>
-            <gaussianNoise>0.0</gaussianNoise>
-            <updateRate>20.0</updateRate>
+            <plugin name="imu_${id}_plugin" filename="libgazebo_ros_imu.so">
+                <alwaysOn>true</alwaysOn>
+                <bodyName>base_link</bodyName>
+                <topicName>imu_${id}</topicName>
+                <serviceName>imu_${id}_service</serviceName>
+                <gaussianNoise>0.0</gaussianNoise>
+                <updateRate>20.0</updateRate>
             </plugin>
         </gazebo>

Commit message: modified for camera and imu

File: calypso_sim/model/auv.urdf.xacro (robot description, xacro)
@@ -48,5 +48,5 @@
       </collision>
       <inertial>
-        <mass value="120"/>
+        <mass value="160"/>
         <inertia ixx="466338.03533197" ixy="0.00022747" ixz="-0.00184206" iyy="846140.53520644" iyz="-13851.49143136" izz="547835.76597596"/>
       </inertial>

File: calypso_sim/model/imu.urdf.xacro (robot description, xacro)
@@ -9,5 +9,4 @@
         <link name="imu_${id}">
             <collision>
-                <origin xyz="0 0 0" rpy="0 0 0"/>
                 <geometry>
                     <box size="0.1 0.1 0.1"/>
@@ -15,5 +14,4 @@
             </collision>
             <visual>
-                <origin xyz="0 0 0" rpy="0 0 0"/>
                 <geometry>
                     <box size="0.1 0.1 0.1"/>
@@ -24,15 +22,17 @@
                 <mass value="0.0001" />
                 <origin xyz="0 0 0" rpy="0 0 ${pi}"/>
-                <inertia ixx="0.0000001" ixy="0" ixz="0" iyy="0.0000001" iyz="0" izz="0.0000001" />
+                <inertia ixx="0.0" ixy="0" ixz="0" iyy="0.0" iyz="0" izz="0.0" />
             </inertial>
         </link>
-        <gazebo reference="imu_${id}_link">
-            <plugin name="imu_${id}_plugin" filename="libgazebo_ros_imu.so">
+=       <gazebo>
+            <plugin name="gazebo_ros_imu_${id}_controller" filename="libgazebo_ros_imu.so">
+                <topicName>/calypso/imu/data</topicName>
+                <serviceName>/calypso/imu/service</serviceName>
+                <bodyName>base_link</bodyName>
+                <gaussianNoise>0</gaussianNoise>
+                <rpyOffsets>0 0 0</rpyOffsets>
+                <updateRate>10.0</updateRate>
                 <alwaysOn>true</alwaysOn>
-                <bodyName>base_link</bodyName>
-                <topicName>imu_${id}</topicName>
-                <serviceName>imu_${id}_service</serviceName>
-                <gaussianNoise>0.0</gaussianNoise>
-                <updateRate>20.0</updateRate>
+                <gaussianNoise>0</gaussianNoise>
             </plugin>
         </gazebo>

Commit message: improved physics plugin

File: calypso_sim/model/auv.urdf.xacro (robot description, xacro)
@@ -48,7 +48,17 @@
       </collision>
       <inertial>
-        <mass value="160"/>
+        <mass value="37"/>
         <inertia ixx="466338.03533197" ixy="0.00022747" ixz="-0.00184206" iyy="846140.53520644" iyz="-13851.49143136" izz="547835.76597596"/>
       </inertial>
+      <fluid>
+        <density>1</density>
+        <origin xyz= "0 0 0"/>
+        <buoyancy>
+            <compensation>1.01</compensation>
+        </buoyancy>
+        <hydrodynamics>
+            <drag xyz="60 100 100" rpy="20 50 50" type="linear"/>
+        </hydrodynamics>
+      </fluid>
     </link>
     <gazebo reference="base_link">
@@ -91,4 +101,5 @@
       </plugin>
     </gazebo>
+<!--
     <gazebo>
       <plugin name="BuoyancyPlugin" filename="libBuoyancyPlugin.so">
@@ -98,4 +109,4 @@
         </link>
       </plugin>
-    </gazebo>
+    </gazebo> -->
 </robot>

File: calypso_sim/model/thrusters.urdf.xacro (robot description, xacro)
@@ -8,5 +8,5 @@
         <material name="red"/>
         <geometry>
-           <mesh filename="${thrusterCCW_path}T200_Thruster.dae" scale="1.5 1.5 1.5"/>
+           <mesh filename="${thrusterCCW_path}T200_Thruster.dae" scale="1 1 1"/>
            <!--<box size="0.1 0.1 0.1"/>-->
         </geometry>
@@ -14,5 +14,5 @@
       <collision>
         <geometry>
-          <mesh filename="${thrusterCCW_path}T200_Thruster.dae" scale="1.5 1.5 1.5"/>
+          <mesh filename="${thrusterCCW_path}T200_Thruster.dae" scale="1 1 1"/>
         </geometry>
       </collision>
@@ -34,10 +34,10 @@
       <visual>
         <geometry>
-          <mesh filename="${thrusterCCW_path}T200_Prop_CCW.dae" scale="1.5 1.5 1.5"/>
-        </geometry>
-      </visual>
-      <collision>
-        <geometry>
-          <mesh filename="${thrusterCCW_path}T200_Prop_CCW.dae" scale="1.5 1.5 1.5"/>
+          <mesh filename="${thrusterCCW_path}T200_Prop_CCW.dae" scale="1 1 1"/>
+        </geometry>
+      </visual>
+      <collision>
+        <geometry>
+          <mesh filename="${thrusterCCW_path}T200_Prop_CCW.dae" scale="1 1 1"/>
         </geometry>
       </collision>
@@ -104,5 +104,5 @@
        <visual>
         <geometry>
-           <mesh filename="${thrusterCW_path}T200_Thruster.dae" scale="1.5 1.5 1.5"/>
+           <mesh filename="${thrusterCW_path}T200_Thruster.dae" scale="1 1 1"/>
            <!--<box size="0.1 0.1 0.1"/>-->
         </geometry>
@@ -111,5 +111,5 @@
       <collision>
         <geometry>
-          <mesh filename="${thrusterCW_path}T200_Thruster.dae" scale="1.5 1.5 1.5"/>
+          <mesh filename="${thrusterCW_path}T200_Thruster.dae" scale="1 1 1"/>
         </geometry>
       </collision>
@@ -131,5 +131,5 @@
       <visual>
         <geometry>
-          <mesh filename="${thrusterCW_path}T200_Prop_CW.dae" scale="1.5 1.5 1.5"/>
+          <mesh filename="${thrusterCW_path}T200_Prop_CW.dae" scale="1 1 1"/>
         </geometry>
         <material name="green"/>
@@ -137,5 +137,5 @@
       <collision>
         <geometry>
-          <mesh filename="${thrusterCW_path}T200_Prop_CW.dae" scale="1.5 1.5 1.5"/>
+          <mesh filename="${thrusterCW_path}T200_Prop_CW.dae" scale="1 1 1"/>
         </geometry>
       </collision>

Commit message: added better bouyancy

File: calypso_sim/model/auv.urdf.xacro (robot description, xacro)
@@ -21,7 +21,7 @@
     <!-- <xacro:property name="x" default="0"/>
     <xacro:property name="y" default="0"/> -->
-    <xacro:property name="x" default="-0.35"/>
-    <xacro:property name="y" default="0.35"/>
-    <xacro:property name="z" default="0"/>
+    <xacro:property name="x" default="-0.26"/>
+    <xacro:property name="y" default="0.43"/>
+    <xacro:property name="z" default="-0.1"/>
     <xacro:property name="r" default="1.57"/>
     <xacro:property name="p" default="0"/>
@@ -37,5 +37,5 @@
         <visual>
           <geometry>
-              <mesh filename="package://calypso_sim/meshes/auv-body/auv.STL" scale="0.001 0.001 0.001"/>
+              <mesh filename="package://calypso_sim/meshes/auv-body/AUV.STL" scale="0.001 0.001 0.001"/>
           </geometry>
           <origin xyz="${x} ${y} ${z}" rpy="${r} ${p} ${Y}" />
@@ -49,16 +49,6 @@
       <inertial>
         <mass value="37"/>
-        <inertia ixx="466338.03533197" ixy="0.00022747" ixz="-0.00184206" iyy="846140.53520644" iyz="-13851.49143136" izz="547835.76597596"/>
+        <inertia ixx="0" ixy="0" ixz="0" iyy="0" iyz="0" izz="0"/>
       </inertial>
-      <fluid>
-        <density>1</density>
-        <origin xyz= "0 0 0"/>
-        <buoyancy>
-            <compensation>1.01</compensation>
-        </buoyancy>
-        <hydrodynamics>
-            <drag xyz="60 100 100" rpy="20 50 50" type="linear"/>
-        </hydrodynamics>
-      </fluid>
     </link>
     <gazebo reference="base_link">
@@ -75,23 +65,23 @@
 -->
     <!-- ${x}-0.32 ${y}-0.06 ${z}+0.1 -->
-    <xacro:thruster_CCW id="1" parent="base_link" xyz="0.26 -0.062 0.1" rpy="0 0 0" axis="0 0 -1">
+    <xacro:thruster_CCW id="1" parent="base_link" xyz="0.185 -0.11 0.1" rpy="0 0 0" axis="0 0 -1">
     </xacro:thruster_CCW>
-    <xacro:thruster_CW id="2" parent="base_link" xyz="${x-x-0.32} ${y-y-0.06} ${z+0.1}" rpy="0 0 0" axis="0 0 1">
+    <xacro:thruster_CW id="2" parent="base_link" xyz="-0.2 -0.11 0.1" rpy="0 0 0" axis="0 0 1">
     </xacro:thruster_CW>
-    <xacro:thruster_CW id="4" parent="base_link" xyz="0.26 0.12 0.1" rpy="0 0 0" axis="0 0 1">
+    <xacro:thruster_CW id="4" parent="base_link" xyz="0.185 0.13 0.1" rpy="0 0 0" axis="0 0 1">
     </xacro:thruster_CW>
-    <xacro:thruster_CCW id="3" parent="base_link" xyz="-0.32 0.12 0.1" rpy="0 0 0" axis="0 0 -1" >
+    <xacro:thruster_CCW id="3" parent="base_link" xyz="-0.2 0.13 0.1" rpy="0 0 0" axis="0 0 -1" >
     </xacro:thruster_CCW>
-    <xacro:thruster_CCW id="5" parent="base_link" xyz="0.22 -0.22 0.06" rpy="0 1.57 0.785" axis="0 0 -1">
+    <xacro:thruster_CCW id="5" parent="base_link" xyz="0.15 -0.25 0.06" rpy="0 1.57 0.785398" axis="0 0 -1">
     </xacro:thruster_CCW>
-    <xacro:thruster_CW id="6" parent="base_link" xyz="-0.23 -0.23 0.06" rpy="0 1.57 2.182" axis="0 0 1">
+    <xacro:thruster_CW id="6" parent="base_link" xyz="-0.15 -0.25 0.06" rpy="0 1.57 2.35619" axis="0 0 1">
     </xacro:thruster_CW>
-    <xacro:thruster_CCW id="7" parent="base_link" xyz="-0.26 0.28 0.06" rpy="0 1.57 3.92" axis="0 0 -1">
+    <xacro:thruster_CCW id="7" parent="base_link" xyz="-0.15 0.25 0.06" rpy="0 1.57 3.92" axis="0 0 -1">
     </xacro:thruster_CCW>
-    <xacro:thruster_CW id="8" parent="base_link" xyz="0.22 0.28 0.06" rpy="0 1.57 -0.785" axis="0 0 1">
+    <xacro:thruster_CW id="8" parent="base_link" xyz="0.15 0.25 0.06" rpy="0 1.57 -0.785398" axis="0 0 1">
     </xacro:thruster_CW>
-    <xacro:camera id="1" parent="base_link" xyz="-0.02 -0.2 0.19" rpy="0 0 -1.57">
+    <xacro:camera id="1" parent="base_link" xyz="-0.005 -0.25 0.13" rpy="0 0 -1.57">
     </xacro:camera>
-    <xacro:imu id="1" parent="base_link" xyz="-0.02 0.1 0.06" rpy="0 0 -1.57">
+    <xacro:imu id="1" parent="base_link" xyz="-0.02 0.1 0.12" rpy="0 0 -1.57">
     </xacro:imu>
     <gazebo>
@@ -101,12 +91,16 @@
       </plugin>
     </gazebo>
-<!--
-    <gazebo>
-      <plugin name="BuoyancyPlugin" filename="libBuoyancyPlugin.so">
-        <fluid_density>1000</fluid_density>
-        <link name="base_link">
-          <volume>0.00964522875</volume>
-        </link>
-      </plugin>
-    </gazebo> -->
+    <plugin name="freebuoyancy_gazebo" filename="libfreebuoyancy_gazebo.so">
+      <descriptionParam>robot_description</descriptionParam>
+      <fluidTopic>current</fluidTopic>
+      <alwaysOn>true</alwaysOn>
+      <surface>0 0 0</surface>
+      <updateRate>.001</updateRate>
+      <link name='base_link'>
+        <buoyancy>
+          <compensation>1.01</compensation>
+          <origin xyz= "0 0 0"/>
+        </buoyancy>
+      </link>
+    </plugin>
 </robot>

File: calypso_sim/model/thrusters.urdf.xacro (robot description, xacro)
@@ -96,4 +96,15 @@
       <allow_auto_disable>0</allow_auto_disable>
     </gazebo>
+    <!-- <gazebo>
+      <plugin name="freefloating_gazebo_control" filename="libfreefloating_gazebo_control.so">
+        <switchService>switch</switchService>
+        <updateRate>100</updateRate>
+        <link>base_link</link>
+        <thruster>
+            <map>${xyz} ${rpy}</map>
+            <effort>30</effort>
+        </thruster>
+      </plugin>
+    </gazebo> -->
      <gazebo reference="prop_${id}">
         <material>Gazebo/Red</material>
@@ -194,6 +205,17 @@
       <allow_auto_disable>0</allow_auto_disable>
     </gazebo>
-     <gazebo reference="prop_${id}">
-        <material>Gazebo/Green</material>
+  <!-- <gazebo>
+      <plugin name="freefloating_gazebo_control" filename="libfreefloating_gazebo_control.so">
+        <switchService>switch</switchService>
+        <updateRate>100</updateRate>
+        <link>base_link</link>
+        <thruster>
+            <map>-1 0 0 0 0 ${-body_width/2}</map>
+            <effort>30</effort>
+        </thruster>
+      </plugin>
+  </gazebo> -->
+    <gazebo reference="prop_${id}">
+      <material>Gazebo/Green</material>
     </gazebo>
   </xacro:macro>

Commit message: fixed massive moving issue

File: calypso_sim/model/auv.urdf.xacro (robot description, xacro)
@@ -23,5 +23,5 @@
     <xacro:property name="x" default="-0.26"/>
     <xacro:property name="y" default="0.43"/>
-    <xacro:property name="z" default="-0.1"/>
+    <xacro:property name="z" default="0"/>
     <xacro:property name="r" default="1.57"/>
     <xacro:property name="p" default="0"/>
@@ -44,11 +44,12 @@
       <collision>
         <geometry>
-          <mesh filename="package://calypso_sim/meshes/auv-body/auv.STL" scale="0.001 0.001 0.001"/>
+          <origin xyz="${x} ${y} ${z}" rpy="${r} ${p} ${Y}" />
+          <mesh filename="package://calypso_sim/meshes/auv-body/AUV.STL" scale="0.001 0.001 0.001"/>
         </geometry>
       </collision>
-      <inertial>
-        <mass value="37"/>
-        <inertia ixx="0" ixy="0" ixz="0" iyy="0" iyz="0" izz="0"/>
-      </inertial>
+    <inertial>
+      <mass value="37.00000000"/>
+      <inertia ixx="1002084.26190628" ixy="-0.00000934" ixz="-0.00004849" iyy="1472890.49211890" iyz="1402.25179064" izz="689649.10160904"/>
+    </inertial>
     </link>
     <gazebo reference="base_link">
@@ -65,24 +66,24 @@
 -->
     <!-- ${x}-0.32 ${y}-0.06 ${z}+0.1 -->
-    <xacro:thruster_CCW id="1" parent="base_link" xyz="0.185 -0.11 0.1" rpy="0 0 0" axis="0 0 -1">
+    <xacro:thruster_CCW id="1" parent="base_link" xyz="0.185 -0.11 0.25" rpy="0 0 0" axis="0 0 -1">
     </xacro:thruster_CCW>
-    <xacro:thruster_CW id="2" parent="base_link" xyz="-0.2 -0.11 0.1" rpy="0 0 0" axis="0 0 1">
+    <xacro:thruster_CW id="2" parent="base_link" xyz="-0.2 -0.11 0.25" rpy="0 0 0" axis="0 0 1">
     </xacro:thruster_CW>
-    <xacro:thruster_CW id="4" parent="base_link" xyz="0.185 0.13 0.1" rpy="0 0 0" axis="0 0 1">
+    <xacro:thruster_CW id="4" parent="base_link" xyz="0.185 0.11 0.25" rpy="0 0 0" axis="0 0 1">
     </xacro:thruster_CW>
-    <xacro:thruster_CCW id="3" parent="base_link" xyz="-0.2 0.13 0.1" rpy="0 0 0" axis="0 0 -1" >
+    <xacro:thruster_CCW id="3" parent="base_link" xyz="-0.2 0.11 0.25" rpy="0 0 0" axis="0 0 -1" >
     </xacro:thruster_CCW>
-    <xacro:thruster_CCW id="5" parent="base_link" xyz="0.15 -0.25 0.06" rpy="0 1.57 0.785398" axis="0 0 -1">
+    <xacro:thruster_CCW id="5" parent="base_link" xyz="0.15 -0.25 0.17" rpy="0 1.57 0.785398" axis="0 0 -1">
     </xacro:thruster_CCW>
-    <xacro:thruster_CW id="6" parent="base_link" xyz="-0.15 -0.25 0.06" rpy="0 1.57 2.35619" axis="0 0 1">
+    <xacro:thruster_CW id="6" parent="base_link" xyz="-0.15 -0.25 0.17" rpy="0 1.57 2.35619" axis="0 0 1">
     </xacro:thruster_CW>
-    <xacro:thruster_CCW id="7" parent="base_link" xyz="-0.15 0.25 0.06" rpy="0 1.57 3.92" axis="0 0 -1">
+    <xacro:thruster_CCW id="7" parent="base_link" xyz="-0.15 0.25 0.17" rpy="0 1.57 3.92" axis="0 0 -1">
     </xacro:thruster_CCW>
-    <xacro:thruster_CW id="8" parent="base_link" xyz="0.15 0.25 0.06" rpy="0 1.57 -0.785398" axis="0 0 1">
+    <xacro:thruster_CW id="8" parent="base_link" xyz="0.15 0.25 0.17" rpy="0 1.57 -0.785398" axis="0 0 1">
     </xacro:thruster_CW>
-    <xacro:camera id="1" parent="base_link" xyz="-0.005 -0.25 0.13" rpy="0 0 -1.57">
+    <!-- <xacro:camera id="1" parent="base_link" xyz="-0.005 -0.25 0.25" rpy="0 0 -1.57">
     </xacro:camera>
-    <xacro:imu id="1" parent="base_link" xyz="-0.02 0.1 0.12" rpy="0 0 -1.57">
-    </xacro:imu>
+    <xacro:imu id="1" parent="base_link" xyz="-0.02 0.1 0.25" rpy="0 0 -1.57">
+    </xacro:imu> -->
     <gazebo>
       <plugin name="gazebo_ros_control" filename="libgazebo_ros_control.so">
@@ -93,5 +94,4 @@
     <plugin name="freebuoyancy_gazebo" filename="libfreebuoyancy_gazebo.so">
       <descriptionParam>robot_description</descriptionParam>
-      <fluidTopic>current</fluidTopic>
       <alwaysOn>true</alwaysOn>
       <surface>0 0 0</surface>
@@ -99,6 +99,6 @@
       <link name='base_link'>
         <buoyancy>
-          <compensation>1.01</compensation>
-          <origin xyz= "0 0 0"/>
+          <compensation>0</compensation>
+          <origin xyz= "${x} ${y} ${z}"/>
         </buoyancy>
       </link>

Commit message: fixed massive moving issue

File: calypso_sim/model/auv.urdf.xacro (robot description, xacro)
@@ -51,4 +51,5 @@
       <mass value="37.00000000"/>
       <inertia ixx="1002084.26190628" ixy="-0.00000934" ixz="-0.00004849" iyy="1472890.49211890" iyz="1402.25179064" izz="689649.10160904"/>
+      <!-- <inertia ixx="0" ixy="0" ixz="0" iyy="0" iyz="0" izz="0"/> -->
     </inertial>
     </link>
@@ -82,8 +83,8 @@
     <xacro:thruster_CW id="8" parent="base_link" xyz="0.15 0.25 0.17" rpy="0 1.57 -0.785398" axis="0 0 1">
     </xacro:thruster_CW>
-    <!-- <xacro:camera id="1" parent="base_link" xyz="-0.005 -0.25 0.25" rpy="0 0 -1.57">
+    <xacro:camera id="1" parent="base_link" xyz="-0.005 -0.25 0.25" rpy="0 0 -1.57">
     </xacro:camera>
     <xacro:imu id="1" parent="base_link" xyz="-0.02 0.1 0.25" rpy="0 0 -1.57">
-    </xacro:imu> -->
+    </xacro:imu>
     <gazebo>
       <plugin name="gazebo_ros_control" filename="libgazebo_ros_control.so">
@@ -100,5 +101,5 @@
         <buoyancy>
           <compensation>0</compensation>
-          <origin xyz= "${x} ${y} ${z}"/>
+          <origin xyz="0 0 0"/>
         </buoyancy>
       </link>
