Commit message: fixing center of mass

File: calypso_sim/model/auv.urdf.xacro (robot description, xacro)
@@ -32,5 +32,5 @@
         <parent link="dummy"/>
         <child link="base_link"/>
-        <origin xyz="${x} ${y} ${z}" rpy="${r} ${p} ${Y}"/>
+        <origin xyz="0 0 0" rpy="${r} ${p} ${Y}"/>
     </joint> -->
     <link name="base_link">
@@ -39,10 +39,10 @@
               <mesh filename="package://calypso_sim/meshes/auv-body/AUV.STL" scale="0.001 0.001 0.001"/>
           </geometry>
-          <origin xyz="${x} ${y} ${z}" rpy="${r} ${p} ${Y}" />
+          <origin xyz="0 0 0" rpy="${r} ${p} ${Y}" />
           <material name="yellow"/>
       </visual>
       <collision>
         <geometry>
-          <origin xyz="${x} ${y} ${z}" rpy="${r} ${p} ${Y}" />
+          <origin xyz="0 0 0" rpy="${r} ${p} ${Y}" />
           <mesh filename="package://calypso_sim/meshes/auv-body/AUV.STL" scale="0.001 0.001 0.001"/>
         </geometry>
@@ -67,23 +67,25 @@
 -->
     <!-- ${x}-0.32 ${y}-0.06 ${z}+0.1 -->
-    <xacro:thruster_CCW id="1" parent="base_link" xyz="0.185 -0.11 0.25" rpy="0 0 0" axis="0 0 -1">
+    <xacro:thruster_CCW id="1" parent="base_link" xyz="0.445 -0.54 0.25" rpy="0 0 0" axis="0 0 -1">
     </xacro:thruster_CCW>
-    <xacro:thruster_CW id="2" parent="base_link" xyz="-0.2 -0.11 0.25" rpy="0 0 0" axis="0 0 1">
+    <xacro:thruster_CW id="2" parent="base_link" xyz="0.06 -0.54 0.25" rpy="0 0 0" axis="0 0 1">
     </xacro:thruster_CW>
-    <xacro:thruster_CW id="4" parent="base_link" xyz="0.185 0.11 0.25" rpy="0 0 0" axis="0 0 1">
+    <xacro:thruster_CW id="4" parent="base_link" xyz="0.445 -0.32 0.25" rpy="0 0 0" axis="0 0 1">
     </xacro:thruster_CW>
-    <xacro:thruster_CCW id="3" parent="base_link" xyz="-0.2 0.11 0.25" rpy="0 0 0" axis="0 0 -1" >
+    <xacro:thruster_CCW id="3" parent="base_link" xyz="0.06 -0.32 0.25" rpy="0 0 0" axis="0 0 -1" >
     </xacro:thruster_CCW>
-    <xacro:thruster_CCW id="5" parent="base_link" xyz="0.15 -0.25 0.17" rpy="0 1.57 0.785398" axis="0 0 -1">
+    <xacro:property name="x" default="-0.26"/>
+    <xacro:property name="y" default="0.43"/>
+    <xacro:thruster_CCW id="5" parent="base_link" xyz="0.41 -0.68 0.17" rpy="0 1.57 0.785398" axis="0 0 -1">
     </xacro:thruster_CCW>
-    <xacro:thruster_CW id="6" parent="base_link" xyz="-0.15 -0.25 0.17" rpy="0 1.57 2.35619" axis="0 0 1">
+    <xacro:thruster_CW id="6" parent="base_link" xyz="0.11 -0.68 0.17" rpy="0 1.57 2.35619" axis="0 0 1">
     </xacro:thruster_CW>
-    <xacro:thruster_CCW id="7" parent="base_link" xyz="-0.15 0.25 0.17" rpy="0 1.57 3.92" axis="0 0 -1">
+    <xacro:thruster_CCW id="7" parent="base_link" xyz="0.11 -0.18 0.17" rpy="0 1.57 3.92" axis="0 0 -1">
     </xacro:thruster_CCW>
-    <xacro:thruster_CW id="8" parent="base_link" xyz="0.15 0.25 0.17" rpy="0 1.57 -0.785398" axis="0 0 1">
+    <xacro:thruster_CW id="8" parent="base_link" xyz="0.41 -0.18 0.17" rpy="0 1.57 -0.785398" axis="0 0 1">
     </xacro:thruster_CW>
-    <xacro:camera id="1" parent="base_link" xyz="-0.005 -0.25 0.25" rpy="0 0 -1.57">
+    <xacro:camera id="1" parent="base_link" xyz="0.255 -0.68 0.25" rpy="0 0 -1.57">
     </xacro:camera>
-    <xacro:imu id="1" parent="base_link" xyz="-0.02 0.1 0.25" rpy="0 0 -1.57">
+    <xacro:imu id="1" parent="base_link" xyz="0.24 -0.4 0.25" rpy="0 0 -1.57">
     </xacro:imu>
     <gazebo>
@@ -93,4 +95,5 @@
       </plugin>
     </gazebo>
+  <gazebo>
     <plugin name="freebuoyancy_gazebo" filename="libfreebuoyancy_gazebo.so">
       <descriptionParam>robot_description</descriptionParam>
@@ -101,7 +104,16 @@
         <buoyancy>
           <compensation>0</compensation>
-          <origin xyz="0 0 0"/>
+          <origin xyz="0 0 1.57"/>
         </buoyancy>
       </link>
     </plugin>
+  </gazebo>
+  <!-- <gazebo>
+     <plugin name="BuoyancyPlugin" filename="libBuoyancyPlugin.so">
+      <fluid_density>1000</fluid_density>
+      <link name="base_link">
+        <volume>0.03</volume>
+      </link>
+    </plugin>
+  </gazebo> -->
 </robot>

Commit message: changed plugins

File: calypso_sim/model/auv.urdf.xacro (robot description, xacro)
@@ -95,5 +95,5 @@
       </plugin>
     </gazebo>
-  <gazebo>
+  <!-- <gazebo>
     <plugin name="freebuoyancy_gazebo" filename="libfreebuoyancy_gazebo.so">
       <descriptionParam>robot_description</descriptionParam>
@@ -104,16 +104,17 @@
         <buoyancy>
           <compensation>0</compensation>
-          <origin xyz="0 0 1.57"/>
+          <origin xyz="0 0 0"/>
         </buoyancy>
       </link>
     </plugin>
-  </gazebo>
-  <!-- <gazebo>
+  </gazebo> -->
+  <gazebo>
      <plugin name="BuoyancyPlugin" filename="libBuoyancyPlugin.so">
       <fluid_density>1000</fluid_density>
       <link name="base_link">
         <volume>0.03</volume>
+        <center_of_volume>0 0 0</center_of_volume>
       </link>
     </plugin>
-  </gazebo> -->
+  </gazebo>
 </robot>

Commit message: changed every fooking thing

File: calypso_sim/model/auv.urdf.xacro (robot description, xacro)
@@ -4,4 +4,5 @@
     <xacro:include filename="$(find calypso_sim)/model/imu.urdf.xacro"/>
     <xacro:include filename="$(find calypso_sim)/model/thrusters.urdf.xacro"/>
+    <xacro:include filename="$(find calypso_sim)/model/chasis.urdf.xacro"/>
     <material name="red">
         <color rgba="1 0 0 1"/>
@@ -27,34 +28,5 @@
     <xacro:property name="p" default="0"/>
     <xacro:property name="Y" default="0"/>
-    <!-- <link name="dummy">
-    </link>
-    <joint name="base_link_to_dummy" type="fixed">
-        <parent link="dummy"/>
-        <child link="base_link"/>
-        <origin xyz="0 0 0" rpy="${r} ${p} ${Y}"/>
-    </joint> -->
-    <link name="base_link">
-        <visual>
-          <geometry>
-              <mesh filename="package://calypso_sim/meshes/auv-body/AUV.STL" scale="0.001 0.001 0.001"/>
-          </geometry>
-          <origin xyz="0 0 0" rpy="${r} ${p} ${Y}" />
-          <material name="yellow"/>
-      </visual>
-      <collision>
-        <geometry>
-          <origin xyz="0 0 0" rpy="${r} ${p} ${Y}" />
-          <mesh filename="package://calypso_sim/meshes/auv-body/AUV.STL" scale="0.001 0.001 0.001"/>
-        </geometry>
-      </collision>
-    <inertial>
-      <mass value="37.00000000"/>
-      <inertia ixx="1002084.26190628" ixy="-0.00000934" ixz="-0.00004849" iyy="1472890.49211890" iyz="1402.25179064" izz="689649.10160904"/>
-      <!-- <inertia ixx="0" ixy="0" ixz="0" iyy="0" iyz="0" izz="0"/> -->
-    </inertial>
-    </link>
-    <gazebo reference="base_link">
-        <material>Gazebo/Yellow</material>
-    </gazebo>
+    <xacro:base_link xyz="0 0 0" rpy="0 1.57 0"></xacro:base_link>
     <!--
 // 2:right upper 1->2
@@ -67,15 +39,13 @@
 -->
     <!-- ${x}-0.32 ${y}-0.06 ${z}+0.1 -->
-    <xacro:thruster_CCW id="1" parent="base_link" xyz="0.445 -0.54 0.25" rpy="0 0 0" axis="0 0 -1">
+    <xacro:thruster_CCW id="1" parent="base_link" xyz="0.25 0.32 -0.17" rpy="0 0 0" axis="0 0 -1">
     </xacro:thruster_CCW>
-    <xacro:thruster_CW id="2" parent="base_link" xyz="0.06 -0.54 0.25" rpy="0 0 0" axis="0 0 1">
+    <xacro:thruster_CW id="2" parent="base_link" xyz="0.25 -0.32 -0.17" rpy="0 0 0" axis="0 0 1">
     </xacro:thruster_CW>
-    <xacro:thruster_CW id="4" parent="base_link" xyz="0.445 -0.32 0.25" rpy="0 0 0" axis="0 0 1">
+    <xacro:thruster_CW id="4" parent="base_link" xyz="-0.25 0.32 -0.17" rpy="0 0 0" axis="0 0 1">
     </xacro:thruster_CW>
-    <xacro:thruster_CCW id="3" parent="base_link" xyz="0.06 -0.32 0.25" rpy="0 0 0" axis="0 0 -1" >
+    <xacro:thruster_CCW id="3" parent="base_link" xyz="-0.25 -0.32 -0.17" rpy="0 0 0" axis="0 0 -1" >
     </xacro:thruster_CCW>
-    <xacro:property name="x" default="-0.26"/>
-    <xacro:property name="y" default="0.43"/>
-    <xacro:thruster_CCW id="5" parent="base_link" xyz="0.41 -0.68 0.17" rpy="0 1.57 0.785398" axis="0 0 -1">
+    <!-- <xacro:thruster_CCW id="5" parent="base_link" xyz="0.41 -0.68 0.17" rpy="0 1.57 0.785398" axis="0 0 -1">
     </xacro:thruster_CCW>
     <xacro:thruster_CW id="6" parent="base_link" xyz="0.11 -0.68 0.17" rpy="0 1.57 2.35619" axis="0 0 1">
@@ -84,8 +54,8 @@
     </xacro:thruster_CCW>
     <xacro:thruster_CW id="8" parent="base_link" xyz="0.41 -0.18 0.17" rpy="0 1.57 -0.785398" axis="0 0 1">
-    </xacro:thruster_CW>
-    <xacro:camera id="1" parent="base_link" xyz="0.255 -0.68 0.25" rpy="0 0 -1.57">
+    </xacro:thruster_CW> -->
+    <xacro:camera id="1" parent="base_link" xyz="0.3 0 0" rpy="0 0 0">
     </xacro:camera>
-    <xacro:imu id="1" parent="base_link" xyz="0.24 -0.4 0.25" rpy="0 0 -1.57">
+    <xacro:imu id="1" parent="base_link" xyz="0 0 0.15" rpy="0 0 -1.57">
     </xacro:imu>
     <gazebo>
@@ -99,9 +69,9 @@
       <descriptionParam>robot_description</descriptionParam>
       <alwaysOn>true</alwaysOn>
-      <surface>0 0 0</surface>
+      <surface>0 0 40</surface>
       <updateRate>.001</updateRate>
       <link name='base_link'>
         <buoyancy>
-          <compensation>0</compensation>
+          <compensation>0.0</compensation>
           <origin xyz="0 0 0"/>
         </buoyancy>
@@ -109,6 +79,6 @@
     </plugin>
   </gazebo>
-  <gazebo>
-     <!-- <plugin name="BuoyancyPlugin" filename="libBuoyancyPlugin.so">
+    <!-- <gazebo>
+     <plugin name="BuoyancyPlugin" filename="libBuoyancyPlugin.so">
       <fluid_density>1000</fluid_density>
       <link name="base_link">

Commit message: added depth camera and 2d camera with aruko markers in the world

File: calypso_sim/model/auv.urdf.xacro (robot description, xacro)
@@ -55,8 +55,147 @@
     <xacro:thruster_CCW id="8" parent="base_link" xyz="-0.45 0.2 0" rpy="0 1.57 0.785398" axis="0 0 -1">
     </xacro:thruster_CCW>
+<!--
     <xacro:camera id="1" parent="base_link" xyz="0.3 0 0" rpy="0 0 0">
-    </xacro:camera>
+    </xacro:camera> -->
     <xacro:imu id="1" parent="base_link" xyz="0 0 0.15" rpy="0 0 -1.57">
     </xacro:imu>
+<!-- this is for the 2d camera in the bottom -->
+    <link name="camera_bottom">
+      <visual>
+        <geometry>
+          <box size="0.05 0.05 0.05"/>
+        </geometry>
+        <material name="red"/>
+      </visual>
+      <collision>
+        <geometry>
+          <box size="0.05 0.05 0.05"/>
+        </geometry>
+      </collision>
+      <inertial>
+        <mass value="1.5"/>
+        <origin xyz="0.0 0.0 0.0" rpy="0 0 0"/>
+        <inertia ixx="0.0" ixy="0.0" ixz="0.0" iyy="0.0" iyz="0.0" izz="0.0"/>
+      </inertial>
+    </link>
+    <joint name="base_link_to_camera_bottom_joint" type="fixed">
+      <parent link="base_link"/>
+      <child link="camera_bottom"/>
+      <origin xyz="0 0 -0.19" rpy="1.57 1.57 0"/>
+    </joint>
+    <joint name="camera_optical_joint_bottom" type="fixed">
+      <parent link="camera_bottom"/>
+      <child link="camera_link_optical_bottom"/>
+      <origin xyz="0 0 0" rpy="${-pi/2} 0 ${-pi/2}"/>
+    </joint>
+    <link name="camera_link_optical_bottom"></link>
+    <gazebo reference="camera_bottom">
+      <material>Gazebo/Red</material>
+      <sensor name="camera" type="camera">
+        <pose> 0 0 0 0 0 0 </pose>
+        <visualize>true</visualize>
+        <update_rate>10</update_rate>
+        <camera>
+          <horizontal_fov>1.089</horizontal_fov>
+          <image>
+            <format>R8G8B8</format>
+            <width>640</width>
+            <height>480</height>
+          </image>
+          <clip>
+            <near>0.05</near>
+            <far>8.0</far>
+          </clip>
+        </camera>
+        <plugin name="camera_controller" filename="libgazebo_ros_camera.so">
+          <frame_name>camera_link_optical_bottom</frame_name>
+          <cameraName>calypso_sim/camera_bottom</cameraName>
+          <imageTopicName>image_raw</imageTopicName>
+        </plugin>
+      </sensor>
+    </gazebo>
+<!-- this is for the depth camera in the front -->
+    <link name="camera_front">
+      <visual>
+        <geometry>
+          <box size="0.05 0.05 0.05"/>
+        </geometry>
+        <material name="red"/>
+      </visual>
+      <collision>
+        <geometry>
+          <box size="0.05 0.05 0.05"/>
+        </geometry>
+      </collision>
+      <inertial>
+        <mass value="1.5"/>
+        <origin xyz="0.0 0.0 0.0" rpy="0 0 0"/>
+        <inertia ixx="0.0" ixy="0.0" ixz="0.0" iyy="0.0" iyz="0.0" izz="0.0"/>
+      </inertial>
+    </link>
+    <joint name="base_link_to_camera_front_joint" type="fixed">
+      <parent link="base_link"/>
+      <child link="camera_front"/>
+      <origin xyz="0.3 0 0" rpy="0 0 0"/>
+    </joint>
+    <joint name="camera_optical_joint_front" type="fixed">
+      <parent link="camera_front"/>
+      <child link="camera_link_optical_front"/>
+      <origin xyz="0 0 0" rpy="${-pi/2} 0 ${-pi/2}"/>
+    </joint>
+    <link name="camera_link_optical_front"></link>
+    <gazebo reference="camera_front">
+      <material>Gazebo/Red</material>
+      <sensor name="camera" type="depth">
+        <pose> 0 0 0 0 0 0 </pose>
+        <visualize>true</visualize>
+        <update_rate>10</update_rate>
+        <camera>
+          <horizontal_fov>1.089</horizontal_fov>
+          <image>
+            <format>B8G8R8</format>
+            <width>640</width>
+            <height>480</height>
+          </image>
+          <clip>
+            <near>0.05</near>
+            <far>8.0</far>
+          </clip>
+        </camera>
+        <plugin name="camera_plugin" filename="libgazebo_ros_openni_kinect.so">
+          <frame_name>camera_link_optical_front</frame_name>
+          <!-- <min_depth>0.1</min_depth>
+          <max_depth>100.0</max_depth> -->
+          <!-- <cameraName>calypso_sim/camera_front</cameraName>
+          <imageTopicName>image_raw</imageTopicName>
+          <depthImageTopicName>/calypso_sim/camera_front/image_raw</depthImageTopicName>
+          <pointCloudTopicName>/calypso_sim/camera_front/points</pointCloudTopicName>
+          <frameName>camera_link</frameName>
+          <pointCloudCutoff>0.5</pointCloudCutoff>
+          <pointCloudCutoffMax>3.0</pointCloudCutoffMax> -->
+          <alwaysOn>true</alwaysOn>
+          <!-- <updateRate>0.0</updateRate> -->
+          <cameraName>calypso_sim/camera_front</cameraName>
+          <imageTopicName>/yash_cam/image_raw</imageTopicName>
+          <!-- <cameraInfoTopicName>camera_info</cameraInfoTopicName> -->
+          <depthImageTopicName>image_raw</depthImageTopicName>
+          <depthImageCameraInfoTopicName>camera_info</depthImageCameraInfoTopicName>
+          <pointCloudTopicName>points</pointCloudTopicName>
+          <!-- <frameName>camera_link</frameName> -->
+          <pointCloudCutoff>0.5</pointCloudCutoff>
+          <pointCloudCutoffMax>3.0</pointCloudCutoffMax>
+          <!-- <distortionK1>0</distortionK1>
+          <distortionK2>0</distortionK2>
+          <distortionK3>0</distortionK3>
+          <distortionT1>0</distortionT1>
+          <distortionT2>0</distortionT2>
+          <CxPrime>0</CxPrime>
+          <Cx>0</Cx>
+          <Cy>0</Cy>
+          <focalLength>0</focalLength>
+          <hackBaseline>0</hackBaseline> -->
+        </plugin>
+      </sensor>
+    </gazebo>
     <gazebo>
       <plugin name="gazebo_ros_control" filename="libgazebo_ros_control.so">
